Commit message: Update model with real dimensions

File: src/tvmd/urdf/Navigator-Def.xacro (robot description, xacro)
@@ -2,25 +2,52 @@
 <robot name="tvmd" xmlns:xacro="http://www.ros.org/wiki/xacro">
 <xacro:macro name="navigator">
-  <link name="base_link">
-    <inertial>
-        <origin xyz="0.023872244589948865 -0.0009500409901555752 0.03522161274068737" rpy="0 0 0"/>
-        <mass value="2.83791501"/>
-        <inertia ixx="0.01210074" iyy="0.01841678" izz="0.02144845" ixy="0.00034820" iyz="-0.00017235" ixz="-0.00023145"/>
-    </inertial>
-    <visual>
+    <link name="base_link">
+        <inertial>
+            <origin xyz="0.023872244589948865 -0.0009500409901555752 0.03522161274068737" rpy="0 0 0"/>
+            <mass value="2.83791501"/>
+            <inertia ixx="0.01210074" iyy="0.01841678" izz="0.02144845" ixy="0.00034820" iyz="-0.00017235" ixz="-0.00023145"/>
+        </inertial>
+        <visual>
+            <origin xyz="0 0 0" rpy="0 0 0"/>
+            <geometry>
+            <mesh filename="package://tvmd/meshes/navigator/NavigatorModule-Sim.stl" scale="0.001 0.001 0.001"/>
+            </geometry>
+            <material name="dark_blue"/>
+        </visual>
+        <collision>
+            <origin xyz="0 0 0.05" rpy="0 0 ${pi/4}"/>
+            <geometry>
+                <!-- <mesh filename="package://tvmd/meshes/navigator/NavigatorModule-Sim.stl" scale="0.001 0.001 0.001"/> -->
+                <box size="0.3 0.3 0.1" />
+            </geometry>
+        </collision>
+        <velocity_decay/>
+    </link>
+    <link name="imu_sensor_link">
+        <collision>
+            <origin xyz="0 0 0" rpy="0 0 0"/>
+            <geometry>
+                <box size="0.02 0.02 0.02"/>
+            </geometry>
+        </collision>
+        <visual>
+            <origin xyz="0 0 0" rpy="0 0 0"/>
+            <geometry>
+                <box size="0.02 0.02 0.02"/>
+            </geometry>
+            <material name="gray"/>
+        </visual>
+        <inertial>
+            <mass value="0.001" />
+            <origin xyz="0 0 0" rpy="0 0 0"/>
+            <inertia ixx="0.00000015" ixy="0" ixz="0" iyy="0.00000015" iyz="0" izz="0.00000015" />
+        </inertial>
+    </link>
+    <joint name="imu_sensor_joint" type="fixed">
+        <axis xyz="0 0 1" />
         <origin xyz="0 0 0" rpy="0 0 0"/>
-        <geometry>
-        <mesh filename="package://tvmd/meshes/navigator/NavigatorModule-Sim.stl" scale="0.001 0.001 0.001"/>
-        </geometry>
-        <material name="dark_blue"/>
-    </visual>
-    <collision>
-        <origin xyz="0 0 0" rpy="0 0 0"/>
-        <geometry>
-        <mesh filename="package://tvmd/meshes/navigator/NavigatorModule-Sim.stl" scale="0.001 0.001 0.001"/>
-        </geometry>
-    </collision>
-    <velocity_decay/>
-  </link>
+        <parent link="base_link"/>
+        <child link="imu_sensor_link"/>
+    </joint>
 </xacro:macro>
 <xacro:macro name="rigid_connection" params="parent child pos_x pos_y pos_z z_psi" >

File: src/tvmd/urdf/Single-Agent-Def.xacro (robot description, xacro)
@@ -6,7 +6,7 @@
   <link name="module${module_id}_body_link">
     <inertial>
-      <origin xyz="0.03950362887818236 0.0002336451659535331 -0.03359920964595942" rpy="0 0 0"/>
-    <mass value="0.50885294"/>
-    <inertia ixx="0.00286197" iyy="0.01669981" izz="0.01760490" ixy="0.00001218" iyz="-0.00000803" ixz="-0.00038649"/>
+      <origin xyz="0.0 0.0 0.0" rpy="0 0 0"/>
+      <mass value="0.50823179"/>
+      <inertia ixx="0.01671968" iyy="0.00290137" izz="0.01758533" ixy="-0.00001217" iyz="-0.00003388" ixz="-0.00000326"/>
     </inertial>
     <visual>
@@ -30,10 +30,10 @@
   <link name="module${module_id}_gimbal_link">
     <inertial>
-      <origin xyz="0.1843065553329719 0.00019186033306794898 -0.0008717237920348236" rpy="0 0 0"/>
+      <origin xyz="0.0 0.0 0.0" rpy="0 0 0"/>
         <mass value="0.03395528"/>
-        <inertia ixx="0.00000159" iyy="0.00031944" izz="0.00031947" ixy="0.0" iyz="-0.00000003" ixz="0.0"/>
+        <inertia ixx="0.00034948" iyy="0.00000164" izz="0.00034950" ixy="0.0" iyz="-0.00000002" ixz="0.0"/>
     </inertial>
     <visual>
-      <origin xyz="0.201475 -0.0 0.0" rpy="0 0 0"/>
+      <origin xyz="0.0 0.0 -0.068" rpy="0 0 0"/>
       <geometry>
         <mesh filename="package://tvmd/meshes/agent/Gimbal_Frame_1.stl" scale="0.001 0.001 0.001"/>
@@ -41,10 +41,10 @@
       <material name="gray"/>
     </visual>
-    <!-- <collision>
-      <origin xyz="0.201475 -0.0 0.0" rpy="0 0 0"/>
+    <collision name='module${module_id}_actuator_collision'>
+      <origin xyz="0 0 0" rpy="${pi/2} 0 0"/>
       <geometry>
-        <mesh filename="package://tvmd/meshes/agent/Gimbal_Frame_1.stl" scale="0.001 0.001 0.001"/>
+        <cylinder length="0.400" radius="0.010"/>
       </geometry>
-    </collision> -->
+    </collision>
   </link>
   <xacro:gz_material joint_name="module${module_id}_gimbal_link" color_name="Gray" />
@@ -53,10 +53,10 @@
   <link name="module${module_id}_actuator_link">
     <inertial>
-      <origin xyz="8.674536786092266e-05 -0.012737509954264759 -0.0036057781438169905" rpy="0 0 0"/>
-        <mass value="0.12541538"/>
-        <inertia ixx="0.00030455" iyy="0.00029933" izz="0.00001545" ixy="-0.00000010" iyz="0.00000437" ixz="-0.00000018"/>
+      <origin xyz="0.0 0.0 0.0" rpy="0 0 0"/>
+        <mass value="0.12540720"/>
+        <inertia ixx="0.00029933" iyy="0.00030455" izz="0.00001575" ixy="-0.00000011" iyz="0.00000018" ixz="-0.00000476"/>
     </inertial>
     <visual>
-      <origin xyz="-0.0005 -0.011 0.0" rpy="0 0 0"/>
+      <origin xyz="0.0 0.0 -0.068" rpy="0 0 0"/>
       <geometry>
         <mesh filename="package://tvmd/meshes/agent/Actuator_1.stl" scale="0.001 0.001 0.001"/>
@@ -64,10 +64,4 @@
       <material name="gray"/>
     </visual>
-    <!-- <collision>
-      <origin xyz="-0.0005 -0.011 0.0" rpy="0 0 0"/>
-      <geometry>
-        <mesh filename="package://tvmd/meshes/agent/Actuator_1.stl" scale="0.001 0.001 0.001"/>
-      </geometry>
-    </collision> -->
   </link>
   <xacro:gz_material joint_name="module${module_id}_actuator_link" color_name="Gray" />
@@ -76,21 +70,21 @@
   <link name="module${module_id}_prop1_link">
     <inertial>
-      <origin xyz="3.216065230847529e-08 -3.6756938827939636e-08 -0.003327345566246087" rpy="0 0 0"/>
+      <origin xyz="0.0 0.0 0.0" rpy="0 0 0"/>
         <mass value="0.00253778"/>
-        <inertia ixx="0.00000005" iyy="0.00000705" izz="0.00000702" ixy="0.0" iyz="0.0" ixz="-0.00000009"/>
+        <inertia ixx="0.00000702" iyy="0.00000005" izz="0.00000705" ixy="0.00000000" iyz="-0.00000009" ixz="0.00000000"/>
     </inertial>
     <visual>
-      <origin xyz="-0.0005 -0.0005 -0.0816" rpy="0 0 0"/>
+      <origin xyz="0.0 0.0 0.0" rpy="${pi/2} 0 0"/>
       <geometry>
-        <mesh filename="package://tvmd/meshes/agent/propeller_9047_1.stl" scale="0.001 0.001 0.001"/>
+        <mesh filename="package://tvmd/meshes/agent/Propeller_9047.stl" scale="0.001 0.001 0.001"/>
       </geometry>
       <material name="yellow"/>
     </visual>
-    <!-- <collision>
-      <origin xyz="-0.0005 -0.0005 -0.0816" rpy="0 0 0"/>
+    <collision name='module${module_id}_rotor_1_collision'>
+      <origin xyz="0 0 0" rpy="0 0 0"/>
       <geometry>
-        <mesh filename="package://tvmd/meshes/agent/propeller_9047_1.stl" scale="0.001 0.001 0.001"/>
+        <cylinder length="0.005" radius="0.12"/>
       </geometry>
-    </collision> -->
+    </collision>
   </link>
   <xacro:gz_material joint_name="module${module_id}_prop1_link" color_name="Yellow" />
@@ -99,21 +93,21 @@
   <link name="module${module_id}_prop2_link">
     <inertial>
-      <origin xyz="3.216065230847529e-08 -3.6756938827939636e-08 -0.003327345566246087" rpy="0 0 0"/>
-        <mass value="0.00253778"/>
-        <inertia ixx="0.00000005" iyy="0.00000705" izz="0.00000702" ixy="0.0" iyz="0.0" ixz="-0.00000009"/>
+      <origin xyz="0.0 0.0 0.0" rpy="0 0 0"/>
+      <mass value="0.00253778"/>
+      <inertia ixx="0.00000702" iyy="0.00000005" izz="0.00000705" ixy="0.00000000" iyz="-0.00000009" ixz="0.00000000"/>
     </inertial>
     <visual>
-      <origin xyz="-0.001 -0.0 0.0746" rpy="0 0 0"/>
+      <origin xyz="0.0 0.0 0.0" rpy="${pi/2} 0 0"/>
       <geometry>
-        <mesh filename="package://tvmd/meshes/agent/propeller_9047_2.stl" scale="0.001 0.001 0.001"/>
+        <mesh filename="package://tvmd/meshes/agent/Propeller_9047.stl" scale="0.001 0.001 0.001"/>
       </geometry>
       <material name="yellow"/>
     </visual>
-    <!-- <collision>
-      <origin xyz="-0.001 -0.0 0.0746" rpy="0 0 0"/>
+    <collision name='module${module_id}_rotor_2_collision'>
+      <origin xyz="0 0 0" rpy="0 0 0"/>
       <geometry>
-        <mesh filename="package://tvmd/meshes/agent/propeller_9047_2.stl" scale="0.001 0.001 0.001"/>
+        <cylinder length="0.005" radius="0.12"/>
       </geometry>
-    </collision> -->
+    </collision>
   </link>
   <xacro:gz_material joint_name="module${module_id}_prop2_link" color_name="Yellow" />
@@ -123,42 +117,42 @@
 <xacro:macro name="body_gimbal_joint" params="module_id">
   <joint name="module${module_id}_body_gimbal_joint" type="revolute">
-    <origin xyz="-0.201475 0.0 0.0" rpy="0 0 0"/>
+    <origin xyz="0.0 0.0 0.068" rpy="0 0 0"/>
     <parent link="module${module_id}_body_link"/>
     <child link="module${module_id}_gimbal_link"/>
-    <axis xyz="-1.0 0.0 0.0"/>
+    <axis xyz="0.0 1.0 0.0"/>
     <limit effort="30000" velocity="10.0" lower="${-pi/2}" upper="${pi/2}" />
-    <dynamics damping="1.000" />
+    <dynamics damping="0.000" />
     <physics>
-      <ode implicit_spring_damper="1" />
+      <ode implicit_spring_damper="0" />
     </physics>
   </joint>
   <xacro:simple_transmission joint_name="module${module_id}_body_gimbal_joint" />
   <xacro:gz_servo joint_name="module${module_id}_body_gimbal_joint"
-    sub_topic="servo_${module_id*2-2}" />
+    sub_topic="servo_${module_id*2-1}" />
 </xacro:macro>
 <!-- X-Servo -->
 <xacro:macro name="gimbal_actuator_joint" params="module_id">
   <joint name="module${module_id}_gimbal_actuator_joint" type="revolute">
-    <origin xyz="0.201975 0.011 0.0" rpy="0 0 0"/>
+    <origin xyz="0.0 0.0 0.0" rpy="0 0 0"/>
     <parent link="module${module_id}_gimbal_link"/>
     <child link="module${module_id}_actuator_link"/>
-    <axis xyz="0.0 -1.0 -0.0"/>
+    <axis xyz="1.0 0.0 0.0"/>
     <limit effort="30000" velocity="10.0" lower="${-pi/6}" upper="${pi/6}" />
-    <dynamics damping="1.000" />
+    <dynamics damping="0.000" />
     <physics>
-      <ode implicit_spring_damper="1" />
+      <ode implicit_spring_damper="0" />
     </physics>
   </joint>
   <xacro:simple_transmission joint_name="module${module_id}_gimbal_actuator_joint" />
   <xacro:gz_servo joint_name="module${module_id}_gimbal_actuator_joint"
-    sub_topic="servo_${module_id*2-1}" />
+    sub_topic="servo_${module_id*2-2}" />
 </xacro:macro>
 <!-- Propellers -->
 <xacro:macro name="actuator_prop1_joint" params="module_id">
   <joint name="module${module_id}_actuator_prop1_joint" type="continuous">
-    <origin xyz="0.0 -0.0105 0.0816" rpy="0 0 0"/>
+    <origin xyz="0.0 0.0 0.0781" rpy="0 0 0"/>
     <parent link="module${module_id}_actuator_link"/>
     <child link="module${module_id}_prop1_link"/>
-    <axis xyz="-0.0 -0.0 -1.0"/>
+    <axis xyz="0.0 0.0 1.0"/>
     <limit effort="30000" velocity="10000.0" lower="-1e+16" upper="1e+16" />
     <!-- <limit lower="-1e+16" upper="1e+16" /> -->
@@ -171,8 +165,8 @@
 <xacro:macro name="actuator_prop2_joint" params="module_id">
   <joint name="module${module_id}_actuator_prop2_joint" type="continuous">
-    <origin xyz="0.0005 -0.011 -0.0746" rpy="0 0 0"/>
+    <origin xyz="0.0 0.0 -0.0781" rpy="0 0 0"/>
     <parent link="module${module_id}_actuator_link"/>
     <child link="module${module_id}_prop2_link"/>
-    <axis xyz="0.0 0.0 1.0"/>
+    <axis xyz="0.0 0.0 -1.0"/>
     <limit effort="30000" velocity="10000.0" lower="-1e+16" upper="1e+16" />
     <!-- <limit lower="-1e+16" upper="1e+16" /> -->

File: src/tvmd/urdf/model.urdf (robot description, URDF)
Before this commit: robot tvmd, 21 links, 20 joints
Links:
- added link imu_sensor_link, mass 0.001; collision box size=0.02 0.02 0.02; visual box size=0.02 0.02 0.02
- link base_link: geometry collision box size=0.3 0.3 0.1; visual mesh filename=package://tvmd/meshes/navigator/NavigatorModule-Sim.stl scale=0.001 0.001 0.001
- link module1_actuator_link: mass 0.12541538 -> 0.12540720
- link module1_body_link: mass 0.50885294 -> 0.50823179
- link module1_gimbal_link: geometry collision cylinder length=0.400 radius=0.010; visual mesh filename=package://tvmd/meshes/agent/Gimbal_Frame_1.stl scale=0.001 0.001 0.001
- link module1_prop1_link: geometry collision cylinder length=0.005 radius=0.12; visual mesh filename=package://tvmd/meshes/agent/Propeller_9047.stl scale=0.001 0.001 0.001
- link module1_prop2_link: geometry collision cylinder length=0.005 radius=0.12; visual mesh filename=package://tvmd/meshes/agent/Propeller_9047.stl scale=0.001 0.001 0.001
- link module2_actuator_link: mass 0.12541538 -> 0.12540720
- link module2_body_link: mass 0.50885294 -> 0.50823179
- link module2_gimbal_link: geometry collision cylinder length=0.400 radius=0.010; visual mesh filename=package://tvmd/meshes/agent/Gimbal_Frame_1.stl scale=0.001 0.001 0.001
- link module2_prop1_link: geometry collision cylinder length=0.005 radius=0.12; visual mesh filename=package://tvmd/meshes/agent/Propeller_9047.stl scale=0.001 0.001 0.001
- link module2_prop2_link: geometry collision cylinder length=0.005 radius=0.12; visual mesh filename=package://tvmd/meshes/agent/Propeller_9047.stl scale=0.001 0.001 0.001
- link module3_actuator_link: mass 0.12541538 -> 0.12540720
- link module3_body_link: mass 0.50885294 -> 0.50823179
- link module3_gimbal_link: geometry collision cylinder length=0.400 radius=0.010; visual mesh filename=package://tvmd/meshes/agent/Gimbal_Frame_1.stl scale=0.001 0.001 0.001
- link module3_prop1_link: geometry collision cylinder length=0.005 radius=0.12; visual mesh filename=package://tvmd/meshes/agent/Propeller_9047.stl scale=0.001 0.001 0.001
- link module3_prop2_link: geometry collision cylinder length=0.005 radius=0.12; visual mesh filename=package://tvmd/meshes/agent/Propeller_9047.stl scale=0.001 0.001 0.001
- link module4_actuator_link: mass 0.12541538 -> 0.12540720
- link module4_body_link: mass 0.50885294 -> 0.50823179
- link module4_gimbal_link: geometry collision cylinder length=0.400 radius=0.010; visual mesh filename=package://tvmd/meshes/agent/Gimbal_Frame_1.stl scale=0.001 0.001 0.001
- link module4_prop1_link: geometry collision cylinder length=0.005 radius=0.12; visual mesh filename=package://tvmd/meshes/agent/Propeller_9047.stl scale=0.001 0.001 0.001
- link module4_prop2_link: geometry collision cylinder length=0.005 radius=0.12; visual mesh filename=package://tvmd/meshes/agent/Propeller_9047.stl scale=0.001 0.001 0.001
Joints:
- added joint imu_sensor_joint: type fixed, parent base_link, child imu_sensor_link, origin xyz=0 0 0 rpy=0 0 0, axis 0 0 1
- joint module1_actuator_prop1_joint: axis -0.0 -0.0 -1.0 -> 0.0 0.0 1.0; origin xyz=0.0 -0.0105 0.0816 rpy=0 0 0 -> xyz=0.0 0.0 0.0781 rpy=0 0 0
- joint module1_actuator_prop2_joint: axis 0.0 0.0 1.0 -> 0.0 0.0 -1.0; origin xyz=0.0005 -0.011 -0.0746 rpy=0 0 0 -> xyz=0.0 0.0 -0.0781 rpy=0 0 0
- joint module1_body_gimbal_joint: axis -1.0 0.0 0.0 -> 0.0 1.0 0.0; origin xyz=-0.201475 0.0 0.0 rpy=0 0 0 -> xyz=0.0 0.0 0.068 rpy=0 0 0
- joint module1_gimbal_actuator_joint: axis 0.0 -1.0 -0.0 -> 1.0 0.0 0.0; origin xyz=0.201975 0.011 0.0 rpy=0 0 0 -> xyz=0.0 0.0 0.0 rpy=0 0 0
- joint module2_actuator_prop1_joint: axis -0.0 -0.0 -1.0 -> 0.0 0.0 1.0; origin xyz=0.0 -0.0105 0.0816 rpy=0 0 0 -> xyz=0.0 0.0 0.0781 rpy=0 0 0
- joint module2_actuator_prop2_joint: axis 0.0 0.0 1.0 -> 0.0 0.0 -1.0; origin xyz=0.0005 -0.011 -0.0746 rpy=0 0 0 -> xyz=0.0 0.0 -0.0781 rpy=0 0 0
- joint module2_body_gimbal_joint: axis -1.0 0.0 0.0 -> 0.0 1.0 0.0; origin xyz=-0.201475 0.0 0.0 rpy=0 0 0 -> xyz=0.0 0.0 0.068 rpy=0 0 0
- joint module2_gimbal_actuator_joint: axis 0.0 -1.0 -0.0 -> 1.0 0.0 0.0; origin xyz=0.201975 0.011 0.0 rpy=0 0 0 -> xyz=0.0 0.0 0.0 rpy=0 0 0
- joint module3_actuator_prop1_joint: axis -0.0 -0.0 -1.0 -> 0.0 0.0 1.0; origin xyz=0.0 -0.0105 0.0816 rpy=0 0 0 -> xyz=0.0 0.0 0.0781 rpy=0 0 0
- joint module3_actuator_prop2_joint: axis 0.0 0.0 1.0 -> 0.0 0.0 -1.0; origin xyz=0.0005 -0.011 -0.0746 rpy=0 0 0 -> xyz=0.0 0.0 -0.0781 rpy=0 0 0
- joint module3_body_gimbal_joint: axis -1.0 0.0 0.0 -> 0.0 1.0 0.0; origin xyz=-0.201475 0.0 0.0 rpy=0 0 0 -> xyz=0.0 0.0 0.068 rpy=0 0 0
- joint module3_gimbal_actuator_joint: axis 0.0 -1.0 -0.0 -> 1.0 0.0 0.0; origin xyz=0.201975 0.011 0.0 rpy=0 0 0 -> xyz=0.0 0.0 0.0 rpy=0 0 0
- joint module4_actuator_prop1_joint: axis -0.0 -0.0 -1.0 -> 0.0 0.0 1.0; origin xyz=0.0 -0.0105 0.0816 rpy=0 0 0 -> xyz=0.0 0.0 0.0781 rpy=0 0 0
- joint module4_actuator_prop2_joint: axis 0.0 0.0 1.0 -> 0.0 0.0 -1.0; origin xyz=0.0005 -0.011 -0.0746 rpy=0 0 0 -> xyz=0.0 0.0 -0.0781 rpy=0 0 0
- joint module4_body_gimbal_joint: axis -1.0 0.0 0.0 -> 0.0 1.0 0.0; origin xyz=-0.201475 0.0 0.0 rpy=0 0 0 -> xyz=0.0 0.0 0.068 rpy=0 0 0
- joint module4_gimbal_actuator_joint: axis 0.0 -1.0 -0.0 -> 1.0 0.0 0.0; origin xyz=0.201975 0.011 0.0 rpy=0 0 0 -> xyz=0.0 0.0 0.0 rpy=0 0 0
- joint rigid_base_link_module1_body_link: origin xyz=-0.215 -0.215 0.068 rpy=0 0 0 -> xyz=0.215 0.215 0.0 rpy=0 0 1.5707963267948966
- joint rigid_base_link_module2_body_link: origin xyz=-0.215 0.215 0.068 rpy=0 0 0 -> xyz=0.215 -0.215 0.0 rpy=0 0 1.5707963267948966
- joint rigid_base_link_module3_body_link: origin xyz=0.215 -0.215 0.068 rpy=0 0 0 -> xyz=-0.215 0.215 0.0 rpy=0 0 0
- joint rigid_base_link_module4_body_link: origin xyz=0.215 0.215 0.068 rpy=0 0 0 -> xyz=-0.215 -0.215 0.0 rpy=0 0 0

File: src/tvmd/urdf/tvmd.xacro (robot description, xacro)
@@ -28,14 +28,13 @@
 <xacro:rigid_connection
   parent="base_link" child="module1_body_link"
-  pos_x="-0.215" pos_y="-0.215" pos_z="0.068" z_psi="0" />
+  pos_x="0.215" pos_y="0.215" pos_z="0.0" z_psi="${pi/2}" />
 <xacro:rigid_connection
   parent="base_link" child="module2_body_link"
-  pos_x="-0.215" pos_y="0.215" pos_z="0.068" z_psi="0" />
+  pos_x="0.215" pos_y="-0.215" pos_z="0.0" z_psi="${pi/2}" />
 <xacro:rigid_connection
   parent="base_link" child="module3_body_link"
-  pos_x="0.215" pos_y="-0.215" pos_z="0.068" z_psi="0" />
+  pos_x="-0.215" pos_y="0.215" pos_z="0.0" z_psi="0" />
 <xacro:rigid_connection
   parent="base_link" child="module4_body_link"
-  pos_x="0.215" pos_y="0.215" pos_z="0.068" z_psi="0" />
-<static>0</static>
+  pos_x="-0.215" pos_y="-0.215" pos_z="0.0" z_psi="0" />
 </robot>
