Commit message: Correct servo angle limit

File: src/tvmd/urdf/Single-Agent-Def.xacro (robot description, xacro)
@@ -121,5 +121,6 @@
     <child link="module${module_id}_gimbal_link"/>
     <axis xyz="0.0 1.0 0.0"/>
-    <limit effort="30000" velocity="10.0" lower="${-pi/2}" upper="${pi/2}" />
+    <!-- <limit effort="30000" velocity="10.0" lower="${-pi/2}" upper="${pi/2}" /> -->
+    <limit effort="30000" velocity="10.0" lower="${-pi/4}" upper="${pi/4}" />
     <dynamics damping="0.000" />
     <physics>
@@ -138,5 +139,6 @@
     <child link="module${module_id}_actuator_link"/>
     <axis xyz="1.0 0.0 0.0"/>
-    <limit effort="30000" velocity="10.0" lower="${-pi/6}" upper="${pi/6}" />
+    <!-- <limit effort="30000" velocity="10.0" lower="${-pi/6}" upper="${pi/6}" /> -->
+    <limit effort="30000" velocity="10.0" lower="-0.349" upper="0.349" />
     <dynamics damping="0.000" />
     <physics>
